Commit message: arm

File: HIMLoco-for-Go2W/resources/robots/zgwsarm/zgwsarm.urdf (robot description, URDF)
Before this commit: robot ZGWSARM, 27 links, 26 joints
Links:
- removed link world
- link ROBOT_ARM_LINK7: geometry collision cylinder length=0.08 radius=0.04; visual mesh filename=./assets/ROBOT_ARM_LINK7.STL
Joints:
- removed joint fixed
